File: ZXCT1009/ZXCT1009.kicad_pcb (KiCad board)
At the start: 2 copper layers, 4 parts, among them U1 ZXCT1009, U2 BP

Commit message: adding terminal
Parts:
- added J1: Screw_Terminal_1x02, Terminal_Blocks:TerminalBlock_Pheonix_MKDS1.5-2pol, F.Cu at (91.8, 39.1)
- added J2: Screw_Terminal_1x02, Terminal_Blocks:TerminalBlock_Pheonix_MKDS1.5-2pol, F.Cu at (108.2, 39.1)
Connections:
- net Vin renamed Net-(J1-Pad1)
- R2 pad 2: Net-(R2-Pad2) -> Net-(J1-Pad2)
- U2 pad 1: (no net) -> Net-(U2-Pad1)
- U2 pad 10: (no net) -> Net-(U2-Pad10)
- U2 pad 11: (no net) -> Net-(U2-Pad11)
- U2 pad 12: (no net) -> Net-(U2-Pad12)
- U2 pad 13: (no net) -> Net-(U2-Pad13)
- U2 pad 14: (no net) -> Net-(U2-Pad14)
- U2 pad 15: (no net) -> Net-(U2-Pad15)
- U2 pad 16: (no net) -> Net-(U2-Pad16)
- U2 pad 17: (no net) -> Net-(U2-Pad17)
- U2 pad 18: (no net) -> Net-(U2-Pad18)
- U2 pad 19: (no net) -> Net-(J1-Pad2)
- U2 pad 2: (no net) -> Net-(U2-Pad2)
- U2 pad 20: (no net) -> Net-(U2-Pad20)
- U2 pad 21: (no net) -> Net-(U2-Pad21)
- U2 pad 22: (no net) -> Net-(U2-Pad22)
- U2 pad 23: (no net) -> Net-(U2-Pad23)
- U2 pad 24: (no net) -> Net-(U2-Pad24)
- U2 pad 25: (no net) -> /Vout
- U2 pad 26: (no net) -> Net-(U2-Pad26)
- U2 pad 27: (no net) -> Net-(U2-Pad27)
- U2 pad 28: (no net) -> Net-(U2-Pad28)
- U2 pad 29: (no net) -> Net-(U2-Pad29)
- U2 pad 3: (no net) -> Net-(U2-Pad3)
- U2 pad 30: (no net) -> Net-(U2-Pad30)
- U2 pad 31: (no net) -> Net-(U2-Pad31)
- U2 pad 32: (no net) -> Net-(U2-Pad32)
- U2 pad 33: (no net) -> Net-(U2-Pad33)
- U2 pad 34: (no net) -> Net-(U2-Pad34)
- U2 pad 35: (no net) -> Net-(U2-Pad35)
- U2 pad 36: (no net) -> Net-(U2-Pad36)
- U2 pad 37: (no net) -> Net-(U2-Pad37)
- U2 pad 39: (no net) -> Net-(J1-Pad2)
- U2 pad 4: (no net) -> Net-(U2-Pad4)
- U2 pad 40: (no net) -> Net-(J1-Pad2)
- U2 pad 5: (no net) -> Net-(U2-Pad5)
- U2 pad 6: (no net) -> Net-(U2-Pad6)
- U2 pad 7: (no net) -> Net-(U2-Pad7)
- U2 pad 8: (no net) -> Net-(U2-Pad8)
- U2 pad 9: (no net) -> Net-(U2-Pad9)
